File: pcb/RaspiOmix.brd (EAGLE design)
At the start: 85 x 56 mm, 53 parts, among them IC1 MCP3424-E/SL, IC2 DS1307

Commit message: Misc
Routing:
- net ADR1: track 7.37 -> 8.96 mm
- net ADR0: track 7.37 -> 8.96 mm
- net VSS: vias 7 -> 15
Other:
- board text added: "rev 1.1.2"
- board text removed: "rev 1.1.1"
Changed lines of the file:
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@@
 <text x="72.39" y="44.29125" size="1.778" layer="25">IO 3</text>
 <text x="39.37" y="10.00125" size="1.27" layer="25">AN 0</text>
-<text x="50.8" y="10.31875" size="1.27" layer="25">AN 1</text>
+<text x="50.8" y="10.00125" size="1.27" layer="25">AN 1</text>
 <text x="68.42125" y="10.00125" size="1.27" layer="25">AN 2</text>
 <text x="80.01" y="10.00125" size="1.27" layer="25">AN 3</text>
@@
 <text x="4.1275" y="37.465" size="1.27" layer="25">DIP0</text>
 <text x="4.1275" y="28.575" size="1.27" layer="25">DIP1</text>
-<text x="41.5925" y="25.4" size="1.4224" layer="25">rev 1.1.1</text>
+<text x="41.5925" y="25.4" size="1.4224" layer="25">rev 1.1.2</text>
 <text x="35.56" y="27.305" size="1.9304" layer="25">RaspiO'Mix</text>
 <text x="22.225" y="24.13" size="1.4224" layer="25">CC-BY-SA </text>
@@
 </element>
 <element name="R22" library="rcl" package="M0805" value="10k 0.1%" x="53.0225" y="13.335" smashed="yes" rot="R270">
-<attribute name="NAME" x="49.68875" y="12.065" size="0.889" layer="25"/>
+<attribute name="NAME" x="48.73625" y="11.7475" size="1.27" layer="25"/>
 <attribute name="VALUE" x="50.4825" y="14.605" size="1.27" layer="27" rot="R270"/>
 </element>
@@
 </element>
 <element name="C9" library="rcl" package="PANASONIC_D" value="220uf" x="6.35" y="44.1325" smashed="yes" rot="R180">
-<attribute name="NAME" x="11.91" y="46.9425" size="1.016" layer="25" rot="R180"/>
+<attribute name="NAME" x="12.545" y="46.3075" size="1.016" layer="25" rot="R180"/>
 <attribute name="VALUE" x="8.1" y="46.1075" size="1.016" layer="27" rot="R180"/>
 </element>
@@
 <contactref element="JP1" pad="2"/>
 <contactref element="U$2" pad="NEG"/>
+<via x="10.16" y="29.21" extent="1-16" drill="0.6"/>
+<via x="41.91" y="33.02" extent="1-16" drill="0.6"/>
+<via x="5.08" y="48.26" extent="1-16" drill="0.6"/>
+<via x="11.43" y="41.91" extent="1-16" drill="0.6"/>
+<via x="31.75" y="19.05" extent="1-16" drill="0.6"/>
+<via x="25.4" y="41.91" extent="1-16" drill="0.6"/>
+<via x="62.865" y="39.37" extent="1-16" drill="0.6"/>
+<via x="37.465" y="50.165" extent="1-16" drill="0.6"/>
 <wire x1="8.89" y1="54.61" x2="9.8425" y2="54.9275" width="0" layer="19" extent="1-1"/>
 <wire x1="66.1035" y1="15.24" x2="66.6725" y2="15.24" width="0" layer="19" extent="1-16"/>
@@
 <contactref element="C28" pad="2"/>
 <wire x1="2.2225" y1="34.925" x2="2.2225" y2="32.385" width="0.3048" layer="16"/>
-<wire x1="12.065" y1="38.735" x2="19.27" y2="38.735" width="0.3048" layer="1"/>
-<via x="12.065" y="38.735" extent="1-16" drill="0.6"/>
+<wire x1="8.89" y1="38.735" x2="19.27" y2="38.735" width="0.3048" layer="1"/>
+<via x="8.89" y="38.735" extent="1-16" drill="0.6"/>
 <wire x1="56.455" y1="12.3825" x2="58.1025" y2="12.3825" width="0.3048" layer="1"/>
 <wire x1="58.1025" y1="12.3825" x2="58.42" y2="12.7" width="0.3048" layer="1"/>
@@
 <wire x1="2.2225" y1="34.925" x2="2.2225" y2="37.7825" width="0.3048" layer="16"/>
 <wire x1="2.2225" y1="37.7825" x2="3.175" y2="38.735" width="0.3048" layer="16"/>
-<wire x1="12.065" y1="38.735" x2="3.175" y2="38.735" width="0.3048" layer="16"/>
+<wire x1="8.89" y1="38.735" x2="3.175" y2="38.735" width="0.3048" layer="16"/>
 <wire x1="3.175" y1="38.735" x2="2.2225" y2="39.6875" width="0.3048" layer="16"/>
 <wire x1="2.2225" y1="39.6875" x2="2.2225" y2="48.5775" width="0.3048" layer="16"/>
@@
 <wire x1="57.445" y1="43.5578" x2="57.445" y2="46.015" width="0.3048" layer="1"/>
 <wire x1="57.445" y1="46.015" x2="58.42" y2="46.99" width="0.3048" layer="1"/>
-<wire x1="60.96" y1="46.99" x2="58.42" y2="46.99" width="0.3048" layer="1"/>
+<wire x1="63.1825" y1="46.99" x2="58.42" y2="46.99" width="0.3048" layer="1"/>
 <contactref element="CON_IO_2" pad="1"/>
-<wire x1="64.31" y1="48.26" x2="62.23" y2="48.26" width="0.3048" layer="1"/>
-<wire x1="62.23" y1="48.26" x2="60.96" y2="46.99" width="0.3048" layer="1"/>
+<wire x1="64.31" y1="48.26" x2="64.4525" y2="48.26" width="0.3048" layer="1"/>
+<wire x1="64.4525" y1="48.26" x2="63.1825" y2="46.99" width="0.3048" layer="1"/>
 <contactref element="CON_IO_1" pad="2"/>
 <wire x1="54.88" y1="48.26" x2="54.9275" y2="48.26" width="0.3048" layer="1"/>
@@
 <contactref element="IC3" pad="16"/>
 <wire x1="75.74" y1="47.4825" x2="75.2475" y2="46.99" width="0.3048" layer="1"/>
-<wire x1="62.5475" y1="46.99" x2="61.9125" y2="46.355" width="0.3048" layer="1"/>
-<wire x1="61.9125" y1="46.355" x2="58.7375" y2="46.355" width="0.3048" layer="1"/>
 <wire x1="58.7375" y1="46.355" x2="58.1025" y2="45.72" width="0.3048" layer="1"/>
 <wire x1="58.1025" y1="45.72" x2="58.1025" y2="43.5653" width="0.3048" layer="1"/>
@@
 <wire x1="75.74" y1="48.26" x2="75.74" y2="47.4825" width="0.3048" layer="1"/>
 <contactref element="CON_IO_2" pad="2"/>
-<wire x1="62.5475" y1="46.99" x2="65.7225" y2="46.99" width="0.3048" layer="1"/>
+<wire x1="58.7375" y1="46.355" x2="65.0875" y2="46.355" width="0.3048" layer="1"/>
 <wire x1="66.31" y1="48.26" x2="66.31" y2="47.5775" width="0.3048" layer="1"/>
-<wire x1="66.31" y1="47.5775" x2="65.7225" y2="46.99" width="0.3048" layer="1"/>
+<wire x1="66.31" y1="47.5775" x2="65.0875" y2="46.355" width="0.3048" layer="1"/>
 <wire x1="75.2475" y1="46.99" x2="66.8975" y2="46.99" width="0.3048" layer="1"/>
 <wire x1="66.8975" y1="46.99" x2="66.31" y2="47.5775" width="0.3048" layer="1"/>
@@
 <wire x1="67.31" y1="12.3825" x2="67.6275" y2="12.065" width="0.3048" layer="16"/>
 <wire x1="67.6275" y1="12.065" x2="67.6275" y2="10.795" width="0.3048" layer="16"/>
+<wire x1="67.6275" y1="10.795" x2="69.215" y2="10.795" width="0.1016" layer="16"/>
 </signal>
 <signal name="ADR1">
@@
 <wire x1="67.6275" y1="13.97" x2="67.6275" y2="15.24" width="0.3048" layer="16"/>
 <via x="63.5" y="13.6525" extent="1-16" drill="0.6" diameter="1.016"/>
+<wire x1="67.6275" y1="15.24" x2="69.215" y2="15.24" width="0.1016" layer="16"/>
 </signal>
 <signal name="AN0">
